File: XpandShield_MK1/MK1_1_2/MK1_1_2.kicad_pcb (KiCad board)
At the start: 2 copper layers, 53.3 x 101.6 mm, 0 parts

Commit message: Updated MK1 PCBs
Routing:
- net (no net): track 1586.9 -> 1620.2 mm, vias 277 -> 321
