File: XpandShield_MK2/MK2_1/MK2_1.sch (KiCad schematic (older format))
At the start: 6 parts, among them P0 R_POT_US, P1 R_POT_US, P2 R_POT_US, P3 R_POT_US, P4 R_POT_US, P5 R_POT_US

Commit message: Updated PCB
Parts:
- added A0: Arduino_Micro, symbol MCU_Module:Arduino_Leonardo
- added R0, R1, R10, R11, R12, R13, R14, R15, R16, R17, R18, R19, R2, R20, R21, R22, R23, R3, R4, R5, R6, R7, R8, R9: R_US, symbol Device:R_US
- added SW0, SW1, SW10, SW11, SW12, SW13, SW14, SW15, SW16, SW17, SW18, SW19, SW2, SW20, SW21, SW22, SW23, SW3, SW4, SW5, SW6, SW7, SW8, SW9: SW_Push, symbol Switch:SW_Push
- added U1, U2, U3: 74HC165, symbol 74xx:74HC165
Connections:
- net labels added: CIPO, D10, D9, SCK
- net labels removed: +5V
- wire segments 37 -> 229
- no-connect marks 0 -> 19
Other:
- moved on the sheet: P0, P1, P2, P3, P4, P5
