File: XpandShield_MK2/MK2_1/MK2_1.kicad_pcb (KiCad board)
At the start: 2 copper layers, 181.6 x 55.2 mm, 10 parts

Commit message: Updated PCB
Routing:
- net (no net): track 3099.5 -> 3108.5 mm

Commit message: Updated Board
Parts:
- added AM0: Arduino-Micro, Custom_SO:Arduino-Micro, F.Cu at (87.6, 48.3)
- added B0: .2_in_Press_Button, Xpand:.2_in_Press_Button, F.Cu at (63.5, 56.5)
- added B0: .2_in_Press_Button, Xpand:.2_in_Press_Button, F.Cu at (101.6, 68.6)
- added B0: .2_in_Press_Button, Xpand:.2_in_Press_Button, F.Cu at (63.5, 71.8)
- added B0: .2_in_Press_Button, Xpand:.2_in_Press_Button, F.Cu at (71.1, 64.1)
- added B0: .2_in_Press_Button, Xpand:.2_in_Press_Button, F.Cu at (55.9, 64.1)
- added B0: .2_in_Press_Button, Xpand:.2_in_Press_Button, F.Cu at (125.1, 68.6)
- added B0: .2_in_Press_Button, Xpand:.2_in_Press_Button, F.Cu at (156.2, 33.0)
- added B0: .2_in_Press_Button, Xpand:.2_in_Press_Button, F.Cu at (163.8, 40.6)
- added B0: .2_in_Press_Button, Xpand:.2_in_Press_Button, F.Cu at (156.2, 45.7)
- added B0: .2_in_Press_Button, Xpand:.2_in_Press_Button, F.Cu at (148.6, 50.8)
- added B0: .2_in_Press_Button, Xpand:.2_in_Press_Button, F.Cu at (148.6, 38.1)
- added B0: .2_in_Press_Button, Xpand:.2_in_Press_Button, F.Cu at (141.0, 43.2)
- added B0: .2_in_Press_Button, Xpand:.2_in_Press_Button, F.Cu at (109.9, 68.6)
- added G0: Big_Thru_Hole, Xpand:Big_Thru_Hole, F.Cu at (175.3, 42.5)
- added G0: Big_Thru_Hole, Xpand:Big_Thru_Hole, F.Cu at (161.3, 70.5)
- added G0: Big_Thru_Hole, Xpand:Big_Thru_Hole, F.Cu at (161.3, 57.8)
- added G0: Big_Thru_Hole, Xpand:Big_Thru_Hole, F.Cu at (151.1, 57.8)
- added G0: Big_Thru_Hole, Xpand:Big_Thru_Hole, F.Cu at (158.1, 27.9)
- added G0: Big_Thru_Hole, Xpand:Big_Thru_Hole, F.Cu at (165.1, 27.9)
- added G0: Big_Thru_Hole, Xpand:Big_Thru_Hole, F.Cu at (168.3, 27.9)
- added G0: Big_Thru_Hole, Xpand:Big_Thru_Hole, F.Cu at (175.3, 27.9)
- added G0: Big_Thru_Hole, Xpand:Big_Thru_Hole, F.Cu at (51.3, 27.9)
- added G0: Big_Thru_Hole, Xpand:Big_Thru_Hole, F.Cu at (44.5, 27.9)
- added G0: Big_Thru_Hole, Xpand:Big_Thru_Hole, F.Cu at (61.5, 27.9)
- added G0: Big_Thru_Hole, Xpand:Big_Thru_Hole, F.Cu at (175.3, 65.2)
- added G0: Big_Thru_Hole, Xpand:Big_Thru_Hole, F.Cu at (54.6, 27.9)
- added G0: Big_Thru_Hole, Xpand:Big_Thru_Hole, F.Cu at (44.5, 40.0)
- added G0: Big_Thru_Hole, Xpand:Big_Thru_Hole, F.Cu at (44.5, 62.6)
- added G0: Big_Thru_Hole, Xpand:Big_Thru_Hole, F.Cu at (68.6, 48.9)
- added G0: Big_Thru_Hole, Xpand:Big_Thru_Hole, F.Cu at (58.4, 48.9)
- added G0: Big_Thru_Hole, Xpand:Big_Thru_Hole, F.Cu at (58.4, 36.2)
- added G0: Big_Thru_Hole, Xpand:Big_Thru_Hole, F.Cu at (68.6, 36.2)
- added G0: Big_Thru_Hole, Xpand:Big_Thru_Hole, F.Cu at (151.1, 70.5)
- added P0: 70mil_Big_Thru_Pad, Xpand:70mil_Big_Thru_Pad, F.Cu at (177.2, 35.1)
- added P0: 70mil_Big_Thru_Pad, Xpand:70mil_Big_Thru_Pad, F.Cu at (136.4, 63.0)
- added P0: 70mil_Big_Thru_Pad, Xpand:70mil_Big_Thru_Pad, F.Cu at (134.1, 63.5)
- added P0: 70mil_Big_Thru_Pad, Xpand:70mil_Big_Thru_Pad, F.Cu at (131.1, 65.5)
- added P0: 70mil_Big_Thru_Pad, Xpand:70mil_Big_Thru_Pad, F.Cu at (129.7, 67.4)
- added P0: 70mil_Big_Thru_Pad, Xpand:70mil_Big_Thru_Pad, F.Cu at (130.2, 69.7)
- added P0: 70mil_Thru_Pad, Xpand:70mil_Thru_Pad, F.Cu at (146.1, 61.0)
- added P0: 70mil_Thru_Pad, Xpand:70mil_Thru_Pad, F.Cu at (146.1, 67.3)
- added P0: 70mil_Thru_Pad, Xpand:70mil_Thru_Pad, F.Cu at (150.5, 67.3)
- added P0: 70mil_Thru_Pad, Xpand:70mil_Thru_Pad, F.Cu at (150.5, 61.0)
- added P0: 70mil_Thru_Pad, Xpand:70mil_Thru_Pad, F.Cu at (69.2, 39.4)
- added P0: 70mil_Big_Thru_Pad, Xpand:70mil_Big_Thru_Pad, F.Cu at (173.4, 70.1)
- added P0: 70mil_Thru_Pad, Xpand:70mil_Thru_Pad, F.Cu at (69.2, 45.7)
- added P0: 70mil_Thru_Pad, Xpand:70mil_Thru_Pad, F.Cu at (73.7, 45.7)
- added P0: 70mil_Thru_Pad, Xpand:70mil_Thru_Pad, F.Cu at (73.7, 39.4)
- added P0: 70mil_Thru_Pad, Xpand:70mil_Thru_Pad, F.Cu at (124.5, 27.9)
- added P0: 70mil_Thru_Pad, Xpand:70mil_Thru_Pad, F.Cu at (121.9, 27.9)
- added P0: 70mil_Thru_Pad, Xpand:70mil_Thru_Pad, F.Cu at (119.4, 27.9)
- added P0: 70mil_Thru_Pad, Xpand:70mil_Thru_Pad, F.Cu at (116.8, 27.9)
- added P0: 70mil_Thru_Pad, Xpand:70mil_Thru_Pad, F.Cu at (114.3, 27.9)
- added P0: 70mil_Thru_Pad, Xpand:70mil_Thru_Pad, F.Cu at (111.8, 27.9)
- added P0: 70mil_Thru_Pad, Xpand:70mil_Thru_Pad, F.Cu at (109.2, 27.9)
- added P0: 70mil_Big_Thru_Pad, Xpand:70mil_Big_Thru_Pad, F.Cu at (177.2, 70.1)
- added P0: 70mil_Thru_Pad, Xpand:70mil_Thru_Pad, F.Cu at (45.7, 25.4)
- added P0: 70mil_Thru_Pad, Xpand:70mil_Thru_Pad, F.Cu at (50.2, 25.4)
- added P0: 70mil_Thru_Pad, Xpand:70mil_Thru_Pad, F.Cu at (55.9, 25.4)
- added P0: 70mil_Thru_Pad, Xpand:70mil_Thru_Pad, F.Cu at (60.3, 25.4)
- added P0: 70mil_Thru_Pad, Xpand:70mil_Thru_Pad, F.Cu at (174.0, 25.4)
- added P0: 70mil_Thru_Pad, Xpand:70mil_Thru_Pad, F.Cu at (169.5, 25.4)
- added P0: 70mil_Thru_Pad, Xpand:70mil_Thru_Pad, F.Cu at (163.8, 25.4)
- added P0: 70mil_Thru_Pad, Xpand:70mil_Thru_Pad, F.Cu at (159.4, 25.4)
- added P0: 70mil_Thru_Pad, Xpand:70mil_Thru_Pad, F.Cu at (153.7, 73.0)
- added P0: 70mil_Thru_Pad, Xpand:70mil_Thru_Pad, F.Cu at (156.2, 73.0)
- added P0: 70mil_Thru_Pad, Xpand:70mil_Thru_Pad, F.Cu at (147.3, 47.0)
- added P0: 70mil_Thru_Pad, Xpand:70mil_Thru_Pad, F.Cu at (158.8, 73.0)
- added P0: 70mil_Thru_Pad, Xpand:70mil_Thru_Pad, F.Cu at (165.1, 66.7)
- added P0: 70mil_Thru_Pad, Xpand:70mil_Thru_Pad, F.Cu at (165.1, 64.1)
- added P0: 70mil_Thru_Pad, Xpand:70mil_Thru_Pad, F.Cu at (165.1, 61.6)
- added P0: 70mil_Thru_Pad, Xpand:70mil_Thru_Pad, F.Cu at (66.0, 33.7)
- added P0: 70mil_Thru_Pad, Xpand:70mil_Thru_Pad, F.Cu at (63.5, 33.7)
- added P0: 70mil_Thru_Pad, Xpand:70mil_Thru_Pad, F.Cu at (61.0, 33.7)
- added P0: 70mil_Thru_Pad, Xpand:70mil_Thru_Pad, F.Cu at (54.6, 45.1)
- added P0: 70mil_Thru_Pad, Xpand:70mil_Thru_Pad, F.Cu at (54.6, 42.5)
- added P0: 70mil_Thru_Pad, Xpand:70mil_Thru_Pad, F.Cu at (54.6, 40.0)
- added P0: 70mil_Thru_Pad, Xpand:70mil_Thru_Pad, F.Cu at (149.2, 45.1)
- added P0: 70mil_Big_Thru_Pad, Xpand:70mil_Big_Thru_Pad, F.Cu at (46.4, 35.1)
- added P0: 70mil_Big_Thru_Pad, Xpand:70mil_Big_Thru_Pad, F.Cu at (42.5, 70.1)
- added P0: 70mil_Big_Thru_Pad, Xpand:70mil_Big_Thru_Pad, F.Cu at (42.5, 35.1)
- added P0: 70mil_Big_Thru_Pad, Xpand:70mil_Big_Thru_Pad, F.Cu at (134.1, 74.2)
- added P0: 70mil_Big_Thru_Pad, Xpand:70mil_Big_Thru_Pad, F.Cu at (136.4, 73.7)
- added P0: 70mil_Big_Thru_Pad, Xpand:70mil_Big_Thru_Pad, F.Cu at (140.8, 69.7)
- added P0: 70mil_Big_Thru_Pad, Xpand:70mil_Big_Thru_Pad, F.Cu at (140.3, 67.4)
- renumbered C3 to C2, C2 to C3
Connections:
- C1 pad 1: (no net) -> D9
- C1 pad 10: (no net) -> Q2
- C1 pad 11: (no net) -> B0
- C1 pad 12: (no net) -> B1
- C1 pad 13: (no net) -> B2
- C1 pad 14: (no net) -> B3
- C1 pad 15: (no net) -> D10
- C1 pad 16: (no net) -> 5V
- C1 pad 2: (no net) -> SCK
- C1 pad 3: (no net) -> B7
- C1 pad 4: (no net) -> B6
- C1 pad 5: (no net) -> B5
- C1 pad 6: (no net) -> B4
- C1 pad 8: (no net) -> GND
- C1 pad 9: (no net) -> Q1
- C2 pad 1: (no net) -> D9
- C2 pad 10: (no net) -> Q3
- C2 pad 11: (no net) -> B8
- C2 pad 12: (no net) -> B9
- C2 pad 13: (no net) -> B10
- C2 pad 14: (no net) -> B11
- C2 pad 15: (no net) -> D10
- C2 pad 16: (no net) -> 5V
- C2 pad 2: (no net) -> SCK
- C2 pad 3: (no net) -> B15
- C2 pad 4: (no net) -> B14
- C2 pad 5: (no net) -> B13
- C2 pad 6: (no net) -> B12
- C2 pad 8: (no net) -> GND
- C2 pad 9: (no net) -> Q2
- C3 pad 1: (no net) -> D9
- C3 pad 10: (no net) -> GND
- C3 pad 11: (no net) -> B16
- C3 pad 12: (no net) -> B17
- C3 pad 13: (no net) -> B18
- C3 pad 14: (no net) -> B19
- C3 pad 15: (no net) -> D10
- C3 pad 16: (no net) -> 5V
- C3 pad 2: (no net) -> SCK
- C3 pad 3: (no net) -> B23
- C3 pad 4: (no net) -> B22
- C3 pad 5: (no net) -> B21
- C3 pad 6: (no net) -> B20
- C3 pad 8: (no net) -> GND
- C3 pad 9: (no net) -> Q3
- REF** pad 1: (no net) -> D10
- REF** pad 2: (no net) -> Q1
- REF** pad 3: (no net) -> GND (x6)
- REF** pad 4: (no net) -> CIPO
- REF** pad 5: (no net) -> 5V
- REF** pad 1: (no net) -> GND (x5)
- REF** pad 2: (no net) -> GND (x5)
- REF** pad 4: (no net) -> GND (x5)
- REF** pad 5: (no net) -> B18
- REF** pad 6: (no net) -> B16
- REF** pad 7: (no net) -> B17
- REF** pad 8: (no net) -> B19
- REF** pad 5: (no net) -> B4
- REF** pad 6: (no net) -> B5
- REF** pad 7: (no net) -> B6
- REF** pad 8: (no net) -> B7
- REF** pad 5: (no net) -> B21
- REF** pad 6: (no net) -> B22
- REF** pad 7: (no net) -> B20
- REF** pad 8: (no net) -> B23
- REF** pad 5: (no net) -> B3
- REF** pad 6: (no net) -> B2
- REF** pad 7: (no net) -> B1
- REF** pad 8: (no net) -> B0
- REF** pad 1: (no net) -> B11
- REF** pad 2: (no net) -> B10
- REF** pad 3: (no net) -> B8
- REF** pad 4: (no net) -> B9
- REF** pad 5: (no net) -> GND
- REF** pad 6: (no net) -> GND
- REF** pad 7: (no net) -> GND
- REF** pad 8: (no net) -> GND
- REF** pad 5: (no net) -> B12
- REF** pad 6: (no net) -> B13
- REF** pad 7: (no net) -> B14
- REF** pad 8: (no net) -> B15
Routing:
- net (no net): track 3108.5 -> 0.00 mm, vias 215 -> 0
- net GND: track 0.00 -> 495.2 mm, vias 0 -> 79
- net 5V: track 0.00 -> 482.2 mm, vias 0 -> 3
- net SCK: track 0.00 -> 134.0 mm, vias 0 -> 8
- net B17: track 0.00 -> 130.6 mm, vias 0 -> 3
- net A3: track 0.00 -> 127.1 mm, vias 0 -> 3
- net A5: track 0.00 -> 122.6 mm, vias 0 -> 3
- net D10: track 0.00 -> 114.9 mm, vias 0 -> 4
- net A1: track 0.00 -> 113.3 mm, vias 0 -> 2
- net B14: track 0.00 -> 102.4 mm, vias 0 -> 1
- net D9: track 0.00 -> 96.8 mm, vias 0 -> 5
- net B15: track 0.00 -> 84.8 mm, vias 0 -> 1
- net B1: track 0.00 -> 80.4 mm, vias 0 -> 2
- net B3: track 0.00 -> 77.6 mm, vias 0 -> 2
- net B0: track 0.00 -> 68.1 mm, vias 0 -> 2
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- added copper zone on B.Cu, net GND
- added copper zone on F.Cu, net GND
Other:
- rule via_min_size: 0.381 -> 0.254
- board text removed: "3v3"
- board text removed: "A0"
- board text removed: "A1"
- board text removed: "A2"
- board text removed: "A3"
- board text removed: "A4"
- board text removed: "A5"
- board text removed: "AREF"
- board text removed: "CIPO/D14"
- board text removed: "D10"
- board text removed: "D11"
- board text removed: "D12"
- board text removed: "D13"
- board text removed: "D16/COPI"
- board text removed: "D17/SS"
- board text removed: "D2/SCL"
- board text removed: "D3/SDA"
- board text removed: "D4"
- board text removed: "D5"
- board text removed: "D6"
- board text removed: "D7"
- board text removed: "D8"
- board text removed: "D9"
- board text removed: "NC"
- board text removed: "RST"
- board text removed: "RX"
- board text removed: "SCK/D15"
- board text removed: "TX"
- board text removed: "VIN"

Commit message: Update MK2 Files
Parts:
- removed the P0 at (129.7, 67.4)
- removed the P0 at (130.2, 69.7)
- removed the P0 at (134.1, 74.2)
- removed the P0 at (136.4, 73.7)
- removed the P0 at (140.8, 69.7)
- removed the P0 at (140.3, 67.4)
- added P0: 70mil_Big_Thru_Pad, Xpand:70mil_Big_Thru_Pad, F.Cu at (129.8, 67.3)
- added P0: 70mil_Big_Thru_Pad, Xpand:70mil_Big_Thru_Pad, F.Cu at (130.3, 69.6)
- added P0: 70mil_Big_Thru_Pad, Xpand:70mil_Big_Thru_Pad, F.Cu at (134.1, 74.0)
- added P0: 70mil_Big_Thru_Pad, Xpand:70mil_Big_Thru_Pad, F.Cu at (136.4, 73.5)
- added P0: 70mil_Big_Thru_Pad, Xpand:70mil_Big_Thru_Pad, F.Cu at (140.7, 69.6)
- added P0: 70mil_Big_Thru_Pad, Xpand:70mil_Big_Thru_Pad, F.Cu at (140.2, 67.3)
- moved G0 0.13 mm to (175.3, 42.7)
- moved G0 0.13 mm to (175.3, 65.0)
- moved G0 0.13 mm to (44.5, 40.1)
- moved G0 0.13 mm to (44.5, 62.5)
Routing:
- net GND: track 495.2 -> 491.9 mm

Commit message: Changed PCB
Parts:
- removed the B0 at (156.2, 33.0)
- removed the B0 at (163.8, 40.6)
- removed the B0 at (156.2, 45.7)
- removed the B0 at (148.6, 50.8)
- removed the B0 at (148.6, 38.1)
- removed the B0 at (141.0, 43.2)
- removed the P0 at (147.3, 47.0)
- removed the P0 at (149.2, 45.1)
- added B0: .2_in_Press_Button, Xpand:.2_in_Press_Button, F.Cu at (163.8, 33.0)
- added B0: .2_in_Press_Button, Xpand:.2_in_Press_Button, F.Cu at (156.2, 50.8)
- added B0: .2_in_Press_Button, Xpand:.2_in_Press_Button, F.Cu at (163.8, 45.7)
- added B0: .2_in_Press_Button, Xpand:.2_in_Press_Button, F.Cu at (171.4, 40.6)
- added B0: .2_in_Press_Button, Xpand:.2_in_Press_Button, F.Cu at (148.6, 43.2)
- added B0: .2_in_Press_Button, Xpand:.2_in_Press_Button, F.Cu at (156.2, 38.1)
- added P0: 70mil_Thru_Pad, Xpand:70mil_Thru_Pad, F.Cu at (133.0, 43.2)
- added P0: 70mil_Thru_Pad, Xpand:70mil_Thru_Pad, F.Cu at (133.0, 45.7)
Routing:
- net B6: track 52.6 -> 63.0 mm, vias 1 -> 2
- net B8: track 24.9 -> 32.5 mm
- net B11: track 16.3 -> 23.9 mm
- net B10: track 11.4 -> 19.1 mm, vias 0 -> 1
- net B9: track 27.6 -> 35.2 mm
- net B7: track 51.4 -> 57.5 mm, vias 1 -> 2
- net GND: track 491.9 -> 487.1 mm, vias 79 -> 78
- net 5V: track 482.0 -> 484.8 mm, vias 3 -> 5
- net B12: track 50.1 -> 52.6 mm
Other:
- net class 5V removed
- net class A0 removed
- net class A1 removed
- net class A2 removed
- net class A3 removed
- net class A4 removed
- net class A5 removed
- net class CIPO removed
- net class COPI removed
- net class Default removed
- net class GND removed
- net class SCK removed
