File: XpandShield_MK1/MK1_3/MK1_3.kicad_pcb (KiCad board)
At the start: 2 copper layers, 53.3 x 101.6 mm, 1 part

Commit message: Updated MK1 PCBs
Routing:
- net (no net): track 1616.6 -> 1605.2 mm

Commit message: Updated MK1_3 board
Routing:
- net (no net): track 1605.2 -> 1600.9 mm, vias 283 -> 281

Commit message: Updated MK1_3 Design
Routing:
- net (no net): track 1600.9 -> 1619.7 mm, vias 281 -> 289
